File: hw/template_25x45.sch (EAGLE design)
At the start: 23 parts, among them J1 GROVE-4P-2.0-3470130P1, J2 GROVE-4P-2.0-3470130P1

Commit message: Small layout improvements
Parts:
- removed R3: 10k, rcl:R-EU_R0603
- C1: value 1u -> (none)
- C9: value 10uF -> (none)
- U$6: value STM32F303C -> STM32F103CXTX; device st:STM32F303C -> st:STM32F103CXTX
Connections:
- removed net BOOT0: R3.2, U$6.BOOT0
- net GND: now also LED1.C, U$6.BOOT0; no longer LED1.A, R3.1
- net LED1: now also U$6.PD1/OSC_OUT; no longer U$6.PC13
- net N$4: now also LED1.A; no longer LED1.C
- net OSC_IN: now also U$6.PD0/OSC_IN; no longer U$6.PF0/OSC_IN
Other:
- note added: "POWER SUPPLY (3.3V)"
- note removed: "POWER SUPPLY"
- moved on the sheet: LED1
Changed lines of the file:
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@@
 <part name="GND34" library="supply1" deviceset="GND" device=""/>
 <part name="+3V5" library="supply1" deviceset="+3V3" device=""/>
-<part name="R3" library="rcl" deviceset="R-EU_" device="R0603" value="10k"/>
 <part name="GND7" library="supply1" deviceset="GND" device=""/>
 <part name="+3V6" library="supply1" deviceset="+3V3" device=""/>
@@
 <part name="J2" library="OPL Eagle Library" deviceset="GROVE-4P-2.0" device="-3470130P1"/>
 <part name="U$2" library="coilcraft" deviceset="LPS4018" device=""/>
-<part name="C1" library="rcl" deviceset="C-EU" device="C1206" value="1u"/>
+<part name="C1" library="rcl" deviceset="C-EU" device="C1206"/>
 <part name="GND1" library="supply" deviceset="GND" device=""/>
 <part name="C2" library="rcl" deviceset="C-EU" device="C0603" value="1u"/>
@@
 <part name="GND4" library="supply" deviceset="GND" device=""/>
 <part name="GND5" library="supply" deviceset="GND" device=""/>
-<part name="C9" library="rcl" deviceset="C-EU" device="C0805" value="10uF"/>
+<part name="C9" library="rcl" deviceset="C-EU" device="C0805"/>
 <part name="GND2" library="supply" deviceset="GND" device=""/>
 <part name="GND3" library="supply" deviceset="GND" device=""/>
 <part name="U$3" library="maxim" deviceset="MAX17501" device=""/>
 <part name="J1" library="OPL Eagle Library" deviceset="GROVE-4P-2.0" device="-3470130P1"/>
-<part name="+3V7" library="supply1" deviceset="+3V3" device=""/>
-<part name="U$6" library="st" deviceset="STM32F303C" device=""/>
+<part name="U$6" library="st" deviceset="STM32F103CX" device="TX"/>
 <part name="FRAME1" library="frames" deviceset="DINA3_L" device=""/>
 <part name="GND13" library="supply" deviceset="GND" device=""/>
@@
 <part name="U$1" library="r2p_pcb" deviceset="PCB_25X45" device=""/>
 <part name="U$5" library="abracon" deviceset="ASD" device=""/>
+<part name="+3V7" library="supply1" deviceset="+3V3" device=""/>
 </parts>
 <sheets>
@@
 <wire x1="147.32" y1="93.98" x2="55.88" y2="93.98" width="0.1524" layer="94"/>
 <wire x1="55.88" y1="93.98" x2="55.88" y2="149.86" width="0.1524" layer="94"/>
-<text x="58.42" y="144.78" size="2.54" layer="94">POWER SUPPLY</text>
+<text x="58.42" y="144.78" size="2.54" layer="94">POWER SUPPLY (3.3V)</text>
 <wire x1="55.88" y1="88.9" x2="147.32" y2="88.9" width="0.1524" layer="94"/>
 <wire x1="147.32" y1="88.9" x2="147.32" y2="48.26" width="0.1524" layer="94"/>
@@
 <instance part="GND34" gate="1" x="129.54" y="231.14"/>
 <instance part="+3V5" gate="G$1" x="93.98" y="180.34"/>
-<instance part="R3" gate="G$1" x="129.54" y="208.28" rot="R90"/>
-<instance part="GND7" gate="1" x="129.54" y="198.12"/>
+<instance part="GND7" gate="1" x="45.72" y="248.92" rot="R180"/>
 <instance part="+3V6" gate="G$1" x="134.62" y="165.1" rot="R270"/>
 <instance part="C3" gate="G$1" x="99.06" y="238.76"/>
@@
 <instance part="C7" gate="G$1" x="124.46" y="71.12"/>
 <instance part="GND22" gate="1" x="124.46" y="63.5"/>
-<instance part="LED1" gate="G$1" x="22.86" y="114.3" rot="R180"/>
+<instance part="LED1" gate="G$1" x="22.86" y="116.84"/>
 <instance part="R1" gate="G$1" x="22.86" y="127" rot="R90"/>
 <instance part="GND16" gate="1" x="81.28" y="10.16"/>
@@
 <instance part="U$3" gate="G$1" x="96.52" y="121.92"/>
 <instance part="J1" gate="J" x="71.12" y="21.59"/>
-<instance part="+3V7" gate="G$1" x="134.62" y="139.7"/>
 <instance part="U$6" gate="G$1" x="55.88" y="205.74"/>
 <instance part="FRAME1" gate="G$1" x="0" y="0"/>
@@
 <instance part="U$1" gate="A" x="27.94" y="22.86"/>
 <instance part="U$5" gate="G$1" x="116.84" y="170.18"/>
+<instance part="+3V7" gate="G$1" x="134.62" y="139.7"/>
 </instances>
 <busses>
@@
 </segment>
 <segment>
-<pinref part="R3" gate="G$1" pin="1"/>
-<pinref part="GND7" gate="1" pin="GND"/>
-<wire x1="129.54" y1="200.66" x2="129.54" y2="203.2" width="0.1524" layer="91"/>
-</segment>
-<segment>
 <pinref part="C3" gate="G$1" pin="2"/>
 <pinref part="GND9" gate="1" pin="GND"/>
@@
 </segment>
 <segment>
-<pinref part="LED1" gate="G$1" pin="A"/>
-<pinref part="GND13" gate="1" pin="GND"/>
-</segment>
-<segment>
 <wire x1="78.74" y1="66.04" x2="76.2" y2="66.04" width="0.1524" layer="91"/>
 <pinref part="GND10" gate="1" pin="GND"/>
 <wire x1="76.2" y1="66.04" x2="76.2" y2="63.5" width="0.1524" layer="91"/>
 <pinref part="SOT1" gate="G$1" pin="RS"/>
+</segment>
+<segment>
+<pinref part="U$6" gate="G$1" pin="BOOT0"/>
+<pinref part="GND7" gate="1" pin="GND"/>
+<wire x1="45.72" y1="246.38" x2="45.72" y2="236.22" width="0.1524" layer="91"/>
+</segment>
+<segment>
+<pinref part="GND13" gate="1" pin="GND"/>
+<pinref part="LED1" gate="G$1" pin="C"/>
 </segment>
 </net>
@@
 <segment>
 <wire x1="63.5" y1="177.8" x2="63.5" y2="175.26" width="0.1524" layer="91"/>
-<label x="63.5" y="170.18" size="1.778" layer="95" rot="R90"/>
+<label x="63.5" y="175.26" size="1.778" layer="95" rot="MR270"/>
 <pinref part="U$6" gate="G$1" pin="PA13"/>
 </segment>
@@
 <segment>
 <wire x1="66.04" y1="177.8" x2="66.04" y2="175.26" width="0.1524" layer="91"/>
-<label x="66.04" y="170.18" size="1.778" layer="95" rot="R90"/>
+<label x="66.04" y="175.26" size="1.778" layer="95" rot="MR270"/>
 <pinref part="U$6" gate="G$1" pin="PA14"/>
 </segment>
@@
 <segment>
 <wire x1="68.58" y1="177.8" x2="68.58" y2="175.26" width="0.1524" layer="91"/>
-<label x="68.58" y="170.18" size="1.778" layer="95" rot="R90"/>
+<label x="68.58" y="175.26" size="1.778" layer="95" rot="MR270"/>
 <pinref part="U$6" gate="G$1" pin="PA15"/>
 </segment>
@@
 </segment>
 <segment>
-<pinref part="U$6" gate="G$1" pin="PC13"/>
-<wire x1="58.42" y1="236.22" x2="58.42" y2="238.76" width="0.1524" layer="91"/>
-<label x="58.42" y="238.76" size="1.778" layer="95" rot="R90"/>
+<wire x1="48.26" y1="236.22" x2="48.26" y2="238.76" width="0.1524" layer="91"/>
+<label x="48.26" y="238.76" size="1.778" layer="95" rot="R90"/>
+<pinref part="U$6" gate="G$1" pin="PD1/OSC_OUT"/>
 </segment>
 </net>
@@
 <wire x1="50.8" y1="236.22" x2="50.8" y2="238.76" width="0.1524" layer="91"/>
 <label x="50.8" y="238.76" size="1.778" layer="95" rot="R90"/>
-<pinref part="U$6" gate="G$1" pin="PF0/OSC_IN"/>
+<pinref part="U$6" gate="G$1" pin="PD0/OSC_IN"/>
 </segment>
 <segment>
@@
 <label x="86.36" y="215.9" size="1.778" layer="95"/>
 <pinref part="U$6" gate="G$1" pin="PB9"/>
-</segment>
-</net>
-<net name="BOOT0" class="0">
-<segment>
-<wire x1="45.72" y1="236.22" x2="45.72" y2="238.76" width="0.1524" layer="91"/>
-<label x="45.72" y="238.76" size="1.778" layer="95" rot="R90"/>
-<pinref part="U$6" gate="G$1" pin="BOOT0"/>
-</segment>
-<segment>
-<wire x1="121.92" y1="215.9" x2="129.54" y2="215.9" width="0.1524" layer="91"/>
-<wire x1="129.54" y1="215.9" x2="129.54" y2="213.36" width="0.1524" layer="91"/>
-<pinref part="R3" gate="G$1" pin="2"/>
-<label x="114.3" y="215.9" size="1.778" layer="95"/>
 </segment>
 </net>
@@
 <segment>
 <pinref part="R1" gate="G$1" pin="1"/>
-<pinref part="LED1" gate="G$1" pin="C"/>
 <wire x1="22.86" y1="119.38" x2="22.86" y2="121.92" width="0.1524" layer="91"/>
-</segment>
-</net>
+<pinref part="LED1" gate="G$1" pin="A"/>
+</segment>
+</net>

Commit message: Updated to R2P Eagle libraries
Parts:
- C1: value (none) -> 1u; device rcl:C-EUC1206 -> r2p_rcl:C-1206
- C14, C17, C2, C3, C4, C6, C7, C8: device rcl:C-EUC0603 -> r2p_rcl:C-0603
- C5: device rcl:C-EUC0805 -> r2p_rcl:C-0805
- C9: value (none) -> 10u; device rcl:C-EUC0805 -> r2p_rcl:C-0805
- J1, J2: value GROVE-4P-2.0-3470130P1 -> R2P_BUS-VERTICAL; device OPL Eagle Library:GROVE-4P-2.0-3470130P1 -> r2p_connector:R2P_BUS-VERTICAL
- LED1: value (none) -> LED0805; device led:LEDCHIPLED_0805 -> r2p_led:LED0805
- R1: device rcl:R-EU_R0603 -> r2p_rcl:R-0603
- SOT1: device maxim:MAX3051EKA -> r2p_ic:MAX3051EKA
- U$2: device coilcraft:LPS4018 -> r2p_rcl:LPS4018
- U$3: device maxim:MAX17501 -> r2p_ic:MAX17501
- U$4: value FTSH-105TH -> JTAG-TH; device samtec:FTSH-105TH -> r2p_connector:JTAG-TH
- U$5: value ASD -> ABRACON_ASD; device abracon:ASD -> r2p_ic:ABRACON_ASD
- U$6: value STM32F103CXTX -> STM32F303CTX; device st:STM32F103CXTX -> r2p_ic:STM32F303CTX
Connections:
- net VIN renamed +VBUS
- net +3V3: now also U$4.1; no longer U$4.P$1
- net GND: now also U$4.3, U$4.5, U$4.7, U$4.9; no longer U$4.P$3, U$4.P$5, U$4.P$7, U$4.P$9
- net JTCK: now also U$4.4; no longer U$4.P$4
- net JTDI: now also U$4.8; no longer U$4.P$8
- net JTDO: now also U$4.6; no longer U$4.P$6
- net JTMS: now also U$4.2; no longer U$4.P$2
- net LED1: now also U$6.PF1/OSC_OUT; no longer U$6.PD1/OSC_OUT
- net NRST: now also U$4.10; no longer U$4.P$10
- net OSC_IN: now also U$6.PF0/OSC_IN; no longer U$6.PD0/OSC_IN

Commit message: Updated keepout
Parts:
- C1: device r2p_rcl:C-1206 -> r2p_rcl:C1206
- C14, C17, C2, C3, C4, C6, C7, C8: device r2p_rcl:C-0603 -> r2p_rcl:C0603
- C5, C9: device r2p_rcl:C-0805 -> r2p_rcl:C0805
- R1: device r2p_rcl:R-0603 -> r2p_rcl:R0603
- U$2: value LPS4018 -> (none)
Changed lines of the file:
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@@
 </classes>
 <parts>
-<part name="C6" library="r2p_rcl" deviceset="C" device="-0603" value="10n"/>
+<part name="C6" library="r2p_rcl" deviceset="C" device="0603" value="10n"/>
 <part name="GND11" library="r2p_supply" deviceset="GND" device=""/>
 <part name="GND12" library="r2p_supply" deviceset="GND" device=""/>
@@
 <part name="GND6" library="r2p_supply" deviceset="GND" device=""/>
 <part name="+3V4" library="r2p_supply" deviceset="+3V3" device=""/>
-<part name="C17" library="r2p_rcl" deviceset="C" device="-0603" value="100n"/>
-<part name="C14" library="r2p_rcl" deviceset="C" device="-0603" value="100n"/>
-<part name="C4" library="r2p_rcl" deviceset="C" device="-0603" value="100n"/>
+<part name="C17" library="r2p_rcl" deviceset="C" device="0603" value="100n"/>
+<part name="C14" library="r2p_rcl" deviceset="C" device="0603" value="100n"/>
+<part name="C4" library="r2p_rcl" deviceset="C" device="0603" value="100n"/>
 <part name="GND29" library="r2p_supply" deviceset="GND" device=""/>
 <part name="GND30" library="r2p_supply" deviceset="GND" device=""/>
 <part name="GND31" library="r2p_supply" deviceset="GND" device=""/>
 <part name="+3V11" library="r2p_supply" deviceset="+3V3" device=""/>
-<part name="C5" library="r2p_rcl" deviceset="C" device="-0805" value="4.7u"/>
+<part name="C5" library="r2p_rcl" deviceset="C" device="0805" value="4.7u"/>
 <part name="GND34" library="r2p_supply" deviceset="GND" device=""/>
 <part name="+3V5" library="r2p_supply" deviceset="+3V3" device=""/>
 <part name="GND7" library="r2p_supply" deviceset="GND" device=""/>
 <part name="+3V6" library="r2p_supply" deviceset="+3V3" device=""/>
-<part name="C3" library="r2p_rcl" deviceset="C" device="-0603" value="100n"/>
+<part name="C3" library="r2p_rcl" deviceset="C" device="0603" value="100n"/>
 <part name="GND9" library="r2p_supply" deviceset="GND" device=""/>
 <part name="+3V3" library="r2p_supply" deviceset="+3V3" device=""/>
 <part name="GND8" library="r2p_supply" deviceset="GND" device=""/>
 <part name="GND10" library="r2p_supply" deviceset="GND" device=""/>
-<part name="C7" library="r2p_rcl" deviceset="C" device="-0603" value="100n"/>
+<part name="C7" library="r2p_rcl" deviceset="C" device="0603" value="100n"/>
 <part name="GND22" library="r2p_supply" deviceset="GND" device=""/>
 <part name="LED1" library="r2p_led" deviceset="LED" device="0805" value=""/>
-<part name="R1" library="r2p_rcl" deviceset="R" device="-0603" value="330"/>
+<part name="R1" library="r2p_rcl" deviceset="R" device="0603" value="330"/>
 <part name="GND16" library="r2p_supply" deviceset="GND" device=""/>
 <part name="GND17" library="r2p_supply" deviceset="GND" device=""/>
@@
 <part name="J2" library="r2p_connector" deviceset="R2P_BUS" device="-VERTICAL"/>
 <part name="U$2" library="r2p_rcl" deviceset="LPS4018" device=""/>
-<part name="C1" library="r2p_rcl" deviceset="C" device="-1206" value="1u"/>
+<part name="C1" library="r2p_rcl" deviceset="C" device="1206" value="1u"/>
 <part name="GND1" library="r2p_supply" deviceset="GND" device=""/>
-<part name="C2" library="r2p_rcl" deviceset="C" device="-0603" value="1u"/>
-<part name="C8" library="r2p_rcl" deviceset="C" device="-0603" value="10n"/>
+<part name="C2" library="r2p_rcl" deviceset="C" device="0603" value="1u"/>
+<part name="C8" library="r2p_rcl" deviceset="C" device="0603" value="10n"/>
 <part name="GND4" library="r2p_supply" deviceset="GND" device=""/>
 <part name="GND5" library="r2p_supply" deviceset="GND" device=""/>
-<part name="C9" library="r2p_rcl" deviceset="C" device="-0805" value="10u"/>
+<part name="C9" library="r2p_rcl" deviceset="C" device="0805" value="10u"/>
 <part name="GND2" library="r2p_supply" deviceset="GND" device=""/>
 <part name="GND3" library="r2p_supply" deviceset="GND" device=""/>
@@
 </segment>
 <segment>
-<wire x1="15.24" y1="60.96" x2="15.24" y2="58.42" width="0.1524" layer="91"/>
+<wire x1="17.78" y1="60.96" x2="15.24" y2="58.42" width="0.1524" layer="91"/>
 <pinref part="U$4" gate="G$1" pin="9"/>
 <pinref part="GND19" gate="1" pin="GND"/>
 <pinref part="U$4" gate="G$1" pin="3"/>
-<wire x1="15.24" y1="68.58" x2="15.24" y2="66.04" width="0.1524" layer="91"/>
-<junction x="15.24" y="60.96"/>
+<wire x1="17.78" y1="68.58" x2="17.78" y2="66.04" width="0.1524" layer="91"/>
+<junction x="17.78" y="60.96"/>
 <pinref part="U$4" gate="G$1" pin="5"/>
-<wire x1="15.24" y1="66.04" x2="15.24" y2="63.5" width="0.1524" layer="91"/>
-<wire x1="15.24" y1="63.5" x2="15.24" y2="60.96" width="0.1524" layer="91"/>
-<junction x="15.24" y="66.04"/>
+<wire x1="17.78" y1="66.04" x2="17.78" y2="63.5" width="0.1524" layer="91"/>
+<wire x1="17.78" y1="63.5" x2="17.78" y2="60.96" width="0.1524" layer="91"/>
+<junction x="17.78" y="66.04"/>
 <pinref part="U$4" gate="G$1" pin="7"/>
-<junction x="15.24" y="63.5"/>
+<junction x="17.78" y="63.5"/>
 </segment>
 <segment>
@@
 </segment>
 <segment>
-<wire x1="15.24" y1="71.12" x2="15.24" y2="73.66" width="0.1524" layer="91"/>
+<wire x1="17.78" y1="71.12" x2="15.24" y2="73.66" width="0.1524" layer="91"/>
 <pinref part="U$4" gate="G$1" pin="1"/>
 <pinref part="+3V1" gate="G$1" pin="+3V3"/>
@@
 </segment>
 <segment>
-<wire x1="35.56" y1="71.12" x2="38.1" y2="71.12" width="0.1524" layer="91"/>
+<wire x1="33.02" y1="71.12" x2="38.1" y2="71.12" width="0.1524" layer="91"/>
 <label x="38.1" y="71.12" size="1.778" layer="95"/>
 <pinref part="U$4" gate="G$1" pin="2"/>
@@
 </segment>
 <segment>
-<wire x1="35.56" y1="68.58" x2="38.1" y2="68.58" width="0.1524" layer="91"/>
+<wire x1="33.02" y1="68.58" x2="38.1" y2="68.58" width="0.1524" layer="91"/>
 <label x="38.1" y="68.58" size="1.778" layer="95"/>
 <pinref part="U$4" gate="G$1" pin="4"/>
@@
 </segment>
 <segment>
-<wire x1="35.56" y1="66.04" x2="38.1" y2="66.04" width="0.1524" layer="91"/>
+<wire x1="33.02" y1="66.04" x2="38.1" y2="66.04" width="0.1524" layer="91"/>
 <label x="38.1" y="66.04" size="1.778" layer="95"/>
 <pinref part="U$4" gate="G$1" pin="6"/>
@@
 </segment>
 <segment>
-<wire x1="35.56" y1="63.5" x2="38.1" y2="63.5" width="0.1524" layer="91"/>
+<wire x1="33.02" y1="63.5" x2="38.1" y2="63.5" width="0.1524" layer="91"/>
 <label x="38.1" y="63.5" size="1.778" layer="95"/>
 <pinref part="U$4" gate="G$1" pin="8"/>
@@
 </segment>
 <segment>
-<wire x1="35.56" y1="60.96" x2="38.1" y2="60.96" width="0.1524" layer="91"/>
+<wire x1="33.02" y1="60.96" x2="38.1" y2="60.96" width="0.1524" layer="91"/>
 <label x="38.1" y="60.96" size="1.778" layer="95"/>
 <pinref part="U$4" gate="G$1" pin="10"/>
